Commit message: 真机遥操

File: fr3c_assets/fr3c_teleop_dual.urdf (robot description, URDF)
Before this commit: robot fr3c_dual, 17 links, 16 joints
Joints:
- joint world_to_left_base: origin xyz=0 0.275 0 rpy=0 0 3.141592653589793 -> xyz=0.0 0.275 0.0 rpy=0 0 1.570796327
- joint world_to_right_base: origin xyz=0 -0.275 0 rpy=0 0 3.141592653589793 -> xyz=0.0 -0.275 0.0 rpy=0 0 1.570796327
